Commit message: fix name and origin of the IMU

File: urdf/anymal.urdf.xacro (robot description, xacro)
@@ -7,6 +7,6 @@
   <xacro:include filename="$(find velodyne_description)/urdf/VLP-16.urdf.xacro" />
   <!-- add the sensors -->
-  <imu name="xsens_mti_100" parent="base">
-    <origin xyz="0.038 0.062 0.184" rpy = "${pi} 0 ${pi}" />
+  <imu name="imu" parent="base">
+    <origin xyz="${0.038+0.02935-0.012} ${0.06245-0.029+0.0229} ${0.1837+0.0095}" rpy = "${pi} 0 ${pi}" />
   </imu>
   <sensor_d435i parent="base" name="realsense_d435i" use_nominal_extrinsics="$(arg simulation)">

File: urdf/xsens_mti.urdf.xacro (robot description, xacro)
@@ -27,7 +27,7 @@
       <xacro:insert_block name="origin" />
       <parent link="${parent}"/>
-      <child link="${name}_base_link"/>
+      <child link="${name}_mount_link"/>
     </joint>
-    <link name="${name}_base_link">
+    <link name="${name}_mount_link">
      <inertial>
         <mass value="0.001" />
@@ -65,8 +65,8 @@
     <joint name="${name}_sensor_joint" type="fixed">
       <origin xyz="${0.02935-0.012} ${.029-.0229} ${0.0095}" rpy="0.0 0.0 0.0" />
-      <parent link="${name}_base_link" />
-      <child link="${name}"/>
+      <parent link="${name}_mount_link" />
+      <child link="${name}_link"/>
     </joint>
-    <link name="${name}"/>
+    <link name="${name}_link"/>
     <material name="${name}_silver">
           <color rgba="0.753 0.753 0.753 1"/>

Commit message: fix origin of the camera

File: urdf/anymal.urdf.xacro (robot description, xacro)
@@ -10,6 +10,22 @@
     <origin xyz="${0.038+0.02935-0.012} ${0.06245-0.029+0.0229} ${0.1837+0.0095}" rpy = "${pi} 0 ${pi}" />
   </imu>
-  <sensor_d435i parent="base" name="realsense_d435i" use_nominal_extrinsics="$(arg simulation)">
-    <origin xyz="0.371 0.018 0.162" rpy="0 ${pi*12.0/180.0} 0" />
+  <!-- fake convenience link representing the optical center of the left camera-->
+  <link name="camera_link" />
+  <!-- this is the joint to update if the camera extrinsics change -->
+  <joint name="base_to_camera_link" type="fixed">
+    <origin xyz="0.371 0.018 0.162" rpy="0 ${pi*11.7/180.0} ${pi*1.75/180.0}" />
+    <parent link="base"/>
+    <child link="camera_link" />
+  </joint>
+  <!-- attachment point for the realsense -->
+  <link name="realsense_parent"/>
+  <!-- this joint brings the camera link back to the bottom screw hole -->
+  <joint name="camera_link_to_parent" type="fixed">
+    <origin xyz="${-0.0149 +0.1e-3 +4.2e-3} -0.0175 ${-0.025/2}" rpy="0 0 0"/>
+    <parent link="camera_link" />
+    <child link="realsense_parent" />
+  </joint>
+  <sensor_d435i parent="realsense_parent" name="realsense_d435i" use_nominal_extrinsics="$(arg simulation)">
+    <origin xyz="0.0 0.0 0.0" rpy="0 0 0" />
   </sensor_d435i>
   <VLP-16 parent="base">

Commit message: add leica tracker prism

File: urdf/anymal.urdf.xacro (robot description, xacro)
@@ -32,3 +32,16 @@
     <origin xyz = "-0.102 0.000 0.290" rpy="0 0 ${-140.0*pi/180.0}" />
   </VLP-16>
+<!-- add Leica prism to be tracked for ground truth -->
+  <link name="leica_prism">
+    <visual>
+      <geometry>
+        <cylinder length="0.03" radius="0.01"/>
+      </geometry>
+    </visual>
+  </link>
+  <joint name="base_to_leica_prism" type="fixed">
+    <origin xyz="-0.037 0 0.355" rpy="0 0 0" />
+    <parent link="base"/>
+    <child link="leica_prism"/>
+  </joint>
 </robot>
